File: x-OSC Programmer.brd (EAGLE design)
At the start: 31.1 x 47 mm, 16 parts

Commit message: Add FTDI header
Parts:
- added H3: RJ11, SparkFun:RJ11-6
- added JP1: (no value), SparkFun:SJ_2S-NO
- H4: value RJ11 -> (none); device SparkFun:RJ11-6 -> SparkFun:1X06
- moved H4 39.4 mm to (6.67, 45.1)
- moved U$1 23.7 mm to (9.53, 18.1)
Connections:
- new net IN1: H1.18, H4.4
- new net N$2: H4.3, JP1.1
- new net OUT1: H2.18, H4.5
- net GND: now also H3.3, H4.1, H4.2; no longer H4.3
- net MCLR: now also H3.1; no longer H4.1
- net PGEC: now also H3.5; no longer H4.5
- net PGED: now also H3.4; no longer H4.4
- net VBATT: now also JP1.2
- net VDD: now also H3.2; no longer H4.2
Routing:
- net N$2: track 0.00 -> 30.9 mm
- net VBATT: track 14.9 -> 32.9 mm
- net MCLR: track 29.1 -> 46.1 mm
- net OUT1: track 0.00 -> 14.7 mm
- net IN1: track 0.00 -> 14.3 mm
- net PGEC: track 16.7 -> 19.2 mm
- net PGED: track 16.2 -> 18.7 mm
Other:
- board text added: "BATT"
- board text added: "IN1"
- board text added: "N/C"
- board text added: "OUT1"
Changed lines of the file:
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@@
 <setting verticaltext="up"/>
 </settings>
-<grid distance="0.025" unitdist="inch" unit="inch" style="dots" multiple="1" display="yes" altdistance="0.000004" altunitdist="inch" altunit="inch"/>
+<grid distance="0.0125" unitdist="inch" unit="inch" style="dots" multiple="1" display="yes" altdistance="0.000004" altunitdist="inch" altunit="inch"/>
 <layers>
 <layer number="1" name="Top" color="4" fill="1" visible="yes" active="yes"/>
@@
 <layer number="43" name="vRestrict" color="2" fill="10" visible="no" active="yes"/>
 <layer number="44" name="Drills" color="7" fill="1" visible="no" active="yes"/>
-<layer number="45" name="Holes" color="7" fill="1" visible="no" active="yes"/>
-<layer number="46" name="Milling" color="3" fill="1" visible="no" active="yes"/>
+<layer number="45" name="Holes" color="7" fill="1" visible="yes" active="yes"/>
+<layer number="46" name="Milling" color="3" fill="1" visible="yes" active="yes"/>
 <layer number="47" name="Measures" color="7" fill="1" visible="no" active="yes"/>
 <layer number="48" name="Document" color="7" fill="1" visible="no" active="yes"/>
@@
 <layer number="122" name="_bsilk" color="7" fill="1" visible="no" active="yes"/>
 <layer number="125" name="_tsilkInv" color="7" fill="1" visible="yes" active="yes"/>
-<layer number="126" name="_bsilkInv" color="7" fill="1" visible="yes" active="yes"/>
+<layer number="126" name="_bsilkInv" color="7" fill="1" visible="no" active="yes"/>
 <layer number="144" name="Drill_legend" color="7" fill="1" visible="no" active="yes"/>
 <layer number="151" name="HeatSink" color="7" fill="1" visible="no" active="yes"/>
@@
 <wire x1="29.5275" y1="0" x2="1.5875" y2="0" width="0" layer="20"/>
 <wire x1="1.5875" y1="0" x2="0" y2="1.5875" width="0" layer="20" curve="-90.007219"/>
-<text x="3.81" y="16.8275" size="1.016" layer="121">x-OSC Programmer v2.0</text>
+<text x="5.08" y="15.5575" size="1.016" layer="121">x-OSC Programmer v2.0</text>
 <text x="15.875" y="26.82875" size="1.016" layer="121">MCLR</text>
 <text x="13.335" y="34.44875" size="1.016" layer="121">SCL</text>
@@
 <text x="7.62" y="37.94125" size="1.016" layer="121" rot="R180">VDD</text>
 <hole x="6.6675" y="22.225" drill="3.1"/>
-<hole x="21.9075" y="42.545" drill="3.1"/>
+<hole x="24.4475" y="42.545" drill="3.1"/>
 <hole x="24.4475" y="14.605" drill="3.1"/>
-<text x="24.4475" y="31.115" size="1.016" layer="121" rot="R180">RESET</text>
-<text x="24.765" y="20.6375" size="1.016" layer="121" rot="R180">POWER</text>
+<text x="25.0825" y="30.7975" size="1.27" layer="121" rot="R180">RESET</text>
+<text x="25.4" y="20.6375" size="1.27" layer="121" rot="R180">POWER</text>
 <wire x1="-0.635" y1="-0.635" x2="31.75" y2="-0.635" width="0" layer="121"/>
 <wire x1="31.75" y1="-0.635" x2="31.75" y2="47.625" width="0" layer="121"/>
 <wire x1="31.75" y1="47.625" x2="-0.635" y2="47.625" width="0" layer="121"/>
 <wire x1="-0.635" y1="47.625" x2="-0.635" y2="-0.635" width="0" layer="121"/>
+<text x="6.19125" y="43.4975" size="1.016" layer="121" rot="R270">GND</text>
+<text x="8.73125" y="43.4975" size="1.016" layer="121" rot="R270">GND</text>
+<text x="11.27125" y="43.4975" size="1.016" layer="121" rot="R270">BATT</text>
+<text x="13.81125" y="43.4975" size="1.016" layer="121" rot="R270">IN1</text>
+<text x="16.35125" y="43.4975" size="1.016" layer="121" rot="R270">OUT1</text>
+<text x="18.89125" y="43.4975" size="1.016" layer="121" rot="R270">N/C</text>
 </plain>
 <attributes>
@@
 <attribute name="VALUE" x="7.9375" y="34.29" size="1.27" layer="27"/>
 </element>
-<element name="H4" library="SparkFun" package="RJ11-6" value="RJ11" x="5.715" y="5.715"/>
+<element name="H3" library="SparkFun" package="RJ11-6" value="RJ11" x="5.715" y="3.175"/>
 <element name="BATT1" library="x-io" package="JST-R/A" value="JST" x="22.86" y="3.81" smashed="yes" rot="R180">
 <attribute name="VALUE" x="24.13" y="3.81" size="0.4064" layer="27" rot="R180"/>
@@
 <attribute name="NAME" x="21.2725" y="38.4175" size="0.8128" layer="25" ratio="10"/>
 </element>
-<element name="U$1" library="x-io" package="X-IO_TECHNOLOGIES_LOGO_8MM_TOP" value="" x="4.7625" y="41.275"/>
+<element name="U$1" library="x-io" package="X-IO_TECHNOLOGIES_LOGO_8MM_TOP" value="" x="9.525" y="18.0975"/>
 <element name="U$2" library="x-io" package="X-OSC_PROGRAMMER_V2.0_SILKSCREEN" value="" x="-0.635" y="-0.635"/>
+<element name="H4" library="SparkFun" package="1X06" value="" x="6.6675" y="45.085" smashed="yes">
+<attribute name="VALUE" x="5.3975" y="41.91" size="1.27" layer="27"/>
+</element>
+<element name="JP1" library="SparkFun" package="SJ_2S-NO" value="" x="16.8275" y="15.875" rot="MR270"/>
 </elements>
 <signals>
 <signal name="GND">
-<contactref element="H4" pad="3"/>
+<contactref element="H3" pad="3"/>
 <contactref element="BATT1" pad="-"/>
 <contactref element="H2" pad="1"/>
@@
 <contactref element="S1" pad="3"/>
 <contactref element="S1" pad="4"/>
+<contactref element="H4" pad="1"/>
+<contactref element="H4" pad="2"/>
 </signal>
 <signal name="PGED">
-<contactref element="H4" pad="4"/>
+<contactref element="H3" pad="4"/>
 <contactref element="P4" pad="1"/>
-<wire x1="11.43" y1="12.065" x2="11.43" y2="25.0825" width="0.254" layer="1"/>
+<wire x1="11.43" y1="9.525" x2="11.43" y2="25.0825" width="0.254" layer="1"/>
 <wire x1="11.43" y1="25.0825" x2="9.2075" y2="27.305" width="0.254" layer="1"/>
 </signal>
 <signal name="PGEC">
-<contactref element="H4" pad="5"/>
+<contactref element="H3" pad="5"/>
 <contactref element="P3" pad="1"/>
-<wire x1="12.7" y1="14.605" x2="12.7" y2="26.3525" width="0.254" layer="1"/>
+<wire x1="12.7" y1="12.065" x2="12.7" y2="26.3525" width="0.254" layer="1"/>
 <wire x1="12.7" y1="26.3525" x2="9.2075" y2="29.845" width="0.254" layer="1"/>
 </signal>
@@
 <wire x1="21.86" y1="10.43" x2="22.225" y2="10.795" width="0.6096" layer="1"/>
 <wire x1="22.225" y1="10.795" x2="24.765" y2="10.795" width="0.6096" layer="1"/>
-<wire x1="24.765" y1="10.795" x2="25.4" y2="10.16" width="0.6096" layer="1"/>
-<wire x1="25.4" y1="10.16" x2="25.4" y2="7.62" width="0.6096" layer="1"/>
-<wire x1="25.4" y1="7.62" x2="27.94" y2="5.08" width="0.6096" layer="1"/>
+<wire x1="24.765" y1="10.795" x2="26.3525" y2="8.89" width="0.6096" layer="1"/>
+<wire x1="26.3525" y1="8.89" x2="26.3525" y2="6.6675" width="0.6096" layer="1"/>
+<wire x1="26.3525" y1="6.6675" x2="27.94" y2="5.08" width="0.6096" layer="1"/>
 <wire x1="29.5275" y1="4.445" x2="28.575" y2="4.445" width="0.6096" layer="1"/>
 <wire x1="28.575" y1="4.445" x2="27.94" y2="5.08" width="0.6096" layer="1"/>
+<wire x1="29.5275" y1="4.445" x2="26.3525" y2="4.445" width="0.6096" layer="16"/>
+<wire x1="26.3525" y1="4.445" x2="16.8275" y2="13.97" width="0.6096" layer="16"/>
+<contactref element="JP1" pad="2"/>
+<wire x1="16.8275" y1="13.97" x2="16.8275" y2="15.425" width="0.6096" layer="16"/>
 </signal>
 <signal name="MCLR">
-<contactref element="H4" pad="1"/>
+<contactref element="H3" pad="1"/>
 <contactref element="P7" pad="1"/>
 <contactref element="S1" pad="1"/>
 <contactref element="S1" pad="2"/>
-<wire x1="7.62" y1="14.605" x2="14.2875" y2="21.2725" width="0.254" layer="16"/>
-<wire x1="14.2875" y1="21.2725" x2="14.2875" y2="27.305" width="0.254" layer="16"/>
-<wire x1="14.2875" y1="27.305" x2="14.2875" y2="28.2956" width="0.254" layer="16"/>
-<wire x1="14.2875" y1="28.2956" x2="18.6563" y2="32.6644" width="0.254" layer="16"/>
-<wire x1="18.6563" y1="32.6644" x2="25.1587" y2="32.6644" width="0.254" layer="16"/>
+<wire x1="7.62" y1="12.065" x2="6.985" y2="11.43" width="0.254" layer="1"/>
+<wire x1="6.985" y1="11.43" x2="6.985" y2="8.89" width="0.254" layer="1"/>
+<wire x1="6.985" y1="8.89" x2="8.255" y2="7.62" width="0.254" layer="1"/>
+<wire x1="8.255" y1="7.62" x2="14.605" y2="7.62" width="0.254" layer="1"/>
+<wire x1="14.605" y1="7.62" x2="15.875" y2="8.89" width="0.254" layer="1"/>
+<wire x1="15.875" y1="8.89" x2="15.875" y2="9.2075" width="0.254" layer="1"/>
+<wire x1="15.875" y1="9.2075" x2="15.875" y2="25.7175" width="0.254" layer="1"/>
+<wire x1="15.875" y1="25.7175" x2="14.2875" y2="27.305" width="0.254" layer="1"/>
+<wire x1="14.2875" y1="27.305" x2="14.2875" y2="28.2956" width="0.254" layer="1"/>
+<wire x1="14.2875" y1="28.2956" x2="18.6563" y2="32.6644" width="0.254" layer="1"/>
+<wire x1="18.6563" y1="32.6644" x2="25.1587" y2="32.6644" width="0.254" layer="1"/>
 </signal>
 <signal name="VDD">
-<contactref element="H4" pad="2"/>
+<contactref element="H3" pad="2"/>
 <contactref element="P1" pad="1"/>
 <contactref element="R1" pad="1"/>
@@
 <wire x1="22.5575" y1="22.325" x2="22.6575" y2="22.225" width="0.254" layer="1"/>
 </signal>
+<signal name="OUT1">
+<contactref element="H4" pad="5"/>
+<contactref element="H2" pad="18"/>
+<wire x1="16.8275" y1="45.085" x2="16.8275" y2="44.45" width="0.254" layer="1"/>
+<wire x1="16.8275" y1="44.45" x2="18.0975" y2="43.18" width="0.254" layer="1"/>
+<wire x1="18.0975" y1="43.18" x2="20.6375" y2="43.18" width="0.254" layer="1"/>
+<wire x1="20.6375" y1="43.18" x2="22.5425" y2="45.085" width="0.254" layer="1"/>
+<wire x1="22.5425" y1="45.085" x2="29.5275" y2="45.085" width="0.254" layer="1"/>
+</signal>
+<signal name="IN1">
+<contactref element="H1" pad="18"/>
+<contactref element="H4" pad="4"/>
+<wire x1="14.2875" y1="45.085" x2="12.3825" y2="43.18" width="0.254" layer="1"/>
+<wire x1="12.3825" y1="43.18" x2="3.4925" y2="43.18" width="0.254" layer="1"/>
+<wire x1="3.4925" y1="43.18" x2="1.5875" y2="45.085" width="0.254" layer="1"/>
+</signal>
+<signal name="N$2">
+<contactref element="H4" pad="3"/>
+<contactref element="JP1" pad="1"/>
+<wire x1="16.8275" y1="16.325" x2="16.8275" y2="40.005" width="0.6096" layer="16"/>
+<wire x1="16.8275" y1="40.005" x2="11.7475" y2="45.085" width="0.6096" layer="16"/>
+</signal>
 </signals>
