File: x-OSC Programmer.sch (EAGLE design)
At the start: 14 parts, among them P1 M01PTH, P2 M01PTH, P3 M01PTH, P4 M01PTH, P5 M01PTH, P6 M01PTH, P7 M01PTH

Commit message: Add FTDI header
Parts:
- added H3: RJ11, SparkFun:RJ11-6PTH
- added JP1: (no value), SparkFun:JUMPER-2SMD-NO
- H4: value RJ11 -> (none); device SparkFun:RJ11-6PTH -> SparkFun:M06SIP
Connections:
- new net IN1: H1.18, H4.4
- new net N$2: H4.3, JP1.1
- new net OUT1: H2.18, H4.5
- net GND: now also H3.3, H4.1, H4.2; no longer H4.3
- net MCLR: now also H3.1; no longer H4.1
- net PGEC: now also H3.5; no longer H4.5
- net PGED: now also H3.4; no longer H4.4
- net VBATT: now also JP1.2
- net VDD: now also H3.2; no longer H4.2
Other:
- note added: "FTDI header"
- moved on the sheet: BATT1, H4, LED1, P1, P2, P3, P4, P5, P6, P7, R1
